Commit message: add existing files

File: src/dual_description/urdf/dual_ur5.urdf.xacro (robot description, xacro)
@@ -7,5 +7,4 @@
     <xacro:arg name="robot_namespace" default="/"/>
     <link name="base_link">
-        <origin rpy="0.0 0 1.5708" xyz="0 0.0 0.0"/>
         <inertial>
             <origin xyz="0 0 0" />
@@ -14,4 +13,5 @@
         </inertial>
         <visual>
+            <origin rpy="1.5708 0.0 3.14159" xyz="0.0 0.0 1.4"/>
             <geometry>
                 <mesh filename="package://dual_description/meshes/STRUCTURE_DAE/structure.dae"/>
